File: PD Charger.kicad_pcb (KiCad board)
At the start: 4 copper layers, 75 x 40 mm, 76 parts, among them J1 USB_C_Receptacle_USB2.0, J2 Conn_ARM_SWD_TagConnect_TC2030, J3 XT60_M, Q1 NMOS, Q2 NMOS, Q3 NMOS, Q4 NMOS, Q5 NTMFS002P03, Q6 NTMFS002P03, Q7 Q_Dual_NMOS_S1G1D2S2G2D1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

Commit message: DRC cleanup and added 3D models
Parts:
- added JP4: SolderJumper_2_Open, Jumper:SolderJumper-2_P1.3mm_Open_RoundedPad1.0x1.5mm, B.Cu at (77.3, 41.5)
- C1: value Cin -> 82u
- C14, C15, C16, C17: value Cin -> 10u
- C18, C19, C20, C21, C27, C28: value Cout -> 10u
- C2: value Cout -> 82u
- C3, C4: value C -> 0.47u
- C34: value FF -> 20p
- R1, R2, R3, R4: value R -> 1
- R10, R7: value Rup -> 100k
- R11: value Rdiv1 -> 36k
- R12: value Rdiv2 -> 9k
- R14, R17: value R -> 100k
- R15: value R -> 752
- R16, R18: value R -> 5820
- moved JP1 1.65 mm to (73.8, 23.0)
Routing:
- net /USB_DP: track 26.6 -> 28.3 mm
- net /USB_DN: track 27.5 -> 28.9 mm
- net Net-(JP1-A): track 1.84 -> 3.28 mm
- net +3V3: track 149.1 -> 149.9 mm
- net VS: vias 71 -> 65
- net GND: vias 146 -> 142
- net /VBUS: vias 30 -> 27

Commit message: export for production
Parts:
- J2: footprint Connector:Tag-Connect_TC2030-IDC-FP_2x03_P1.27mm_Vertical -> Connector:Tag-Connect_TC2030-IDC-NL_2x03_P1.27mm_Vertical
- moved J2 1.54 mm to (82.3, 39.5), turned to 90 degrees
Routing:
- net /SWO: track 20.4 -> 11.3 mm
- net VD: track 96.6 -> 88.2 mm
- net VS: track 59.1 -> 53.7 mm
- net +3V3: track 149.9 -> 153.8 mm
- net /~{RST}: track 30.7 -> 34.4 mm
- net /SWCLK: track 11.6 -> 9.05 mm
- net /FB: track 47.2 -> 46.2 mm

Commit message: silkscreen and testpoints
Parts:
- added C37: 1u, Capacitor_SMD:C_0603_1608Metric, F.Cu at (55.5, 40.0)
- added R21: 33k, Resistor_SMD:R_0603_1608Metric, F.Cu at (29.5, 48.8)
- added SW1: SW_MEC_5G, Button_Switch_SMD:SW_SPST_B3U-1000P-B, F.Cu at (79.8, 45.0)
- added TP1: TestPoint_Small, TestPoint:TestPoint_Pad_D1.0mm, F.Cu at (40.8, 21.5)
- added TP2: TestPoint_Small, TestPoint:TestPoint_Pad_D1.0mm, F.Cu at (45.8, 25.0)
- added TP3: TestPoint_Small, TestPoint:TestPoint_Pad_D1.0mm, F.Cu at (31.3, 40.0)
- added TP4: TestPoint_Small, TestPoint:TestPoint_Pad_D1.0mm, F.Cu at (29.8, 35.0)
- added TP5: TestPoint_Small, TestPoint:TestPoint_Pad_D1.0mm, F.Cu at (49.8, 35.0)
- added TP6: TestPoint_Small, TestPoint:TestPoint_Pad_D1.0mm, F.Cu at (50.3, 40.5)
- added TP7: TestPoint_Small, TestPoint:TestPoint_Pad_D1.0mm, F.Cu at (44.9, 49.3)
- added TP8: TestPoint_Small, TestPoint:TestPoint_Pad_D1.0mm, F.Cu at (79.3, 17.0)
- added TP9: TestPoint_Small, TestPoint:TestPoint_Pad_D1.0mm, F.Cu at (48.3, 40.5)
- moved R7 2.66 mm to (29.5, 47.0), turned to 0 degrees
- moved R8 1.59 mm to (50.7, 43.5)
Connections:
- R7 pad 1: VDD -> VS
Routing:
- net +3V3: track 153.8 -> 128.1 mm
- net VS: track 53.7 -> 60.4 mm
- net VDD: track 10.4 -> 4.76 mm
- net /SYNC: track 34.6 -> 38.7 mm
- net /EN: track 19.9 -> 22.4 mm
- net Net-(U3-TG2): track 7.86 -> 9.80 mm
- net /FB: track 46.2 -> 48.1 mm
- net Net-(U3-BG2): track 7.66 -> 9.53 mm
- net Net-(U3-BG1): track 7.92 -> 9.76 mm
- net Net-(U3-TG1): track 8.12 -> 9.51 mm
- net VD: track 88.2 -> 89.4 mm, vias 16 -> 17
- net /RT: track 9.30 -> 8.30 mm
- net GND: vias 142 -> 160
Other:
- board text added: "Daniel Raymond/FPV Static USBC PD Charger"
