File: KiCad/input.kicad_sch (KiCad schematic)
At the start: 23 parts, among them Q7 SiR5607DP, Q8 SiR5607DP, U5 ADM1270ACPZ, U6 INA293A2

Commit message: new layout
Parts:
- C44, C45, C46, C47, C48: footprint (none) -> Capacitor_SMD:C_0603_1608Metric
- NT5: footprint (none) -> NetTie:NetTie-2_SMD_Pad0.5mm
- R24, R28, R29, R30, R31, R32, R33, R34, R35, R36, R37, R38: footprint (none) -> Resistor_SMD:R_0603_1608Metric
- R25: footprint Resistor_THT:R_Axial_Shunt_L22.2mm_W8.0mm_PS14.30mm_P25.40mm -> Resistor_SMD:R_Shunt_Ohmite_LVK12
Connections:
- net Q7_S: now also R25.1; no longer R25.4
- net Q8_S: now also R25.4; no longer R25.1
- net SENSE+: now also R25.2; no longer R25.3
- net SENSE-: now also R25.3; no longer R25.2
- net ENABLE renamed SOURCE_EN
Other:
- moved on the sheet: R25
Changed lines of the file:
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@@
 	(wire
 		(pts
-			(xy 128.27 115.57) (xy 135.89 115.57)
+			(xy 124.46 115.57) (xy 135.89 115.57)
 		)
 		(stroke
@@
 		)
 	)
-	(label "ENABLE"
-		(at 128.27 115.57 0)
-		(fields_autoplaced yes)
-		(effects
-			(font
-				(size 1.27 1.27)
-			)
-			(justify left bottom)
-		)
-	)
 	(label "VIN"
 		(at 123.19 81.28 0)
@@
 			)
 			(justify right bottom)
+		)
+	)
+	(label "SOURCE_EN"
+		(at 124.46 115.57 0)
+		(fields_autoplaced yes)
+		(effects
+			(font
+				(size 1.27 1.27)
+			)
+			(justify left bottom)
 		)
 	)
@@
 		)
 	)
-	(hierarchical_label "ENABLE"
+	(hierarchical_label "SOURCE_EN"
 		(shape input)
 		(at 139.7 106.68 180)
@@
 			)
 		)
-		(property "Footprint" ""
+		(property "Footprint" "Resistor_SMD:R_0603_1608Metric"
 			(at 184.658 86.36 90)
 			(effects
@@
 			)
 		)
-		(property "Footprint" ""
+		(property "Footprint" "Resistor_SMD:R_0603_1608Metric"
 			(at 173.228 132.08 90)
 			(effects
@@
 			)
 		)
-		(property "Footprint" ""
+		(property "Footprint" "Resistor_SMD:R_0603_1608Metric"
 			(at 119.888 85.09 90)
 			(effects
@@
 			)
 		)
-		(property "Footprint" ""
+		(property "Footprint" "Resistor_SMD:R_0603_1608Metric"
 			(at 130.81 110.998 90)
 			(effects
@@
 			)
 		)
-		(property "Footprint" ""
+		(property "Footprint" "Capacitor_SMD:C_0603_1608Metric"
 			(at 119.0752 111.76 0)
 			(effects
@@
 			)
 		)
-		(property "Footprint" ""
+		(property "Footprint" "Resistor_SMD:R_0603_1608Metric"
 			(at 128.778 92.71 90)
 			(effects
@@
 			)
 		)
-		(property "Footprint" ""
+		(property "Footprint" "Resistor_SMD:R_0603_1608Metric"
 			(at 159.258 135.89 90)
 			(effects
@@
 			)
 		)
-		(property "Footprint" ""
+		(property "Footprint" "Resistor_SMD:R_0603_1608Metric"
 			(at 128.778 85.09 90)
 			(effects
@@
 			)
 		)
-		(property "Footprint" ""
+		(property "Footprint" "Capacitor_SMD:C_0603_1608Metric"
 			(at 148.59 140.6652 0)
 			(effects
@@
 			)
 		)
-		(property "Footprint" ""
+		(property "Footprint" "Resistor_SMD:R_0603_1608Metric"
 			(at 184.658 93.98 90)
 			(effects
@@
 			)
 		)
-		(property "Footprint" ""
+		(property "Footprint" "Resistor_SMD:R_0603_1608Metric"
 			(at 149.098 135.89 90)
 			(effects
@@
 			)
 		)
-		(property "Footprint" ""
+		(property "Footprint" "Capacitor_SMD:C_0603_1608Metric"
 			(at 173.6852 116.84 0)
 			(effects
@@
 			)
 		)
-		(property "Footprint" ""
+		(property "Footprint" "NetTie:NetTie-2_SMD_Pad0.5mm"
 			(at 157.48 58.42 0)
 			(effects
@@
 			)
 		)
-		(property "Footprint" ""
+		(property "Footprint" "Capacitor_SMD:C_0603_1608Metric"
 			(at 181.3052 116.84 0)
 			(effects
@@
 			)
 		)
-		(property "Footprint" ""
+		(property "Footprint" "Capacitor_SMD:C_0603_1608Metric"
 			(at 139.3952 166.37 0)
 			(effects
@@
 			)
 		)
-		(property "Footprint" ""
+		(property "Footprint" "Resistor_SMD:R_0603_1608Metric"
 			(at 183.388 132.08 90)
 			(effects
@@
 			)
 		)
-		(property "Footprint" ""
+		(property "Footprint" "Resistor_SMD:R_0603_1608Metric"
 			(at 137.668 119.38 90)
 			(effects
@@
 			)
 		)
-		(property "Footprint" ""
+		(property "Footprint" "Resistor_SMD:R_0603_1608Metric"
 			(at 184.658 101.6 90)
 			(effects
@@
 	(symbol
 		(lib_id "Device:R_Shunt")
-		(at 147.32 68.58 270)
-		(unit 1)
-		(exclude_from_sim no)
-		(in_bom yes)
-		(on_board yes)
-		(dnp no)
-		(fields_autoplaced yes)
+		(at 147.32 68.58 90)
+		(mirror x)
+		(unit 1)
+		(exclude_from_sim no)
+		(in_bom yes)
+		(on_board yes)
+		(dnp no)
 		(property "Reference" "R25"
 			(at 147.32 62.23 90)
@@
 			)
 		)
-		(property "Footprint" "Resistor_THT:R_Axial_Shunt_L22.2mm_W8.0mm_PS14.30mm_P25.40mm"
+		(property "Footprint" "Resistor_SMD:R_Shunt_Ohmite_LVK12"
 			(at 147.32 66.802 90)
 			(effects

Commit message: standalone regulator core
Parts:
- added TP11, TP12, TP13, TP14, TP15, TP16: TestPoint, TestPoint:TestPoint_Pad_D1.0mm, symbol Connector:TestPoint
Connections:
- net FB_PG: now also TP14.1
- net FLB: now also TP13.1
- net G_BP: now also TP16.1
- net G_RP: now also TP15.1
- net OV: now also TP12.1
- net UV: now also TP11.1
- net SGOOD renamed PGOOD
- net SOURCE_EN renamed ENABLE
