File: KiCad/mcu.kicad_sch (KiCad schematic)
At the start: 15 parts, among them J2 Conn_ARM_SWD_TagConnect_TC2030, SW1 SW_MEC_5G, SW2 SW_MEC_5G, U4 STM32G431CBUx

Commit message: new layout
Connections:
- net ICTRL: now also U4.13 (PA5); no longer U4.12 (PA4)
- net IDMON: now also U4.15 (PA7); no longer U4.19 (PB2)
- net ISMON: now also U4.24 (PB11); no longer U4.18 (PB1)
- net LOAD_DISCHRG: now also U4.2 (PC13); no longer U4.39 (PC10)
- net SYNC: now also U4.47 (PB9); no longer U4.17 (PB0)
- net VCTRL: now also U4.12 (PA4); no longer U4.10 (PA2)
- net VDMON: now also U4.14 (PA6); no longer U4.9 (PA1)
- net VSMON: now also U4.16 (PC4); no longer U4.8 (PA0)
- net UART_RX: now reaches U4.11 (PA3)
- net REG_ON: now reaches U4.25 (PB12)
- net ~{PGOOD}: now reaches U4.26 (PB13)
- net SGOOD: now reaches U4.27 (PB14)
- net ~{FAULT}: now reaches U4.28 (PB15)
- net LOAD_EN: now reaches U4.3 (PC14)
- net SOURCE_EN: now reaches U4.4 (PC15)
- net LOADEN: no longer names the net of U4.40 (PC11)
- new net UART_TX: U4.10 (PA2)
- no-connect marks 17 -> 13
Changed lines of the file:
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@@
 	)
 	(no_connect
-		(at 118.11 123.19)
+		(at 118.11 87.63)
 	)
 	(no_connect
@@
 	)
 	(no_connect
-		(at 118.11 130.81)
-	)
-	(no_connect
-		(at 118.11 128.27)
-	)
-	(no_connect
-		(at 118.11 133.35)
-	)
-	(no_connect
 		(at 118.11 118.11)
-	)
-	(no_connect
-		(at 118.11 90.17)
-	)
-	(no_connect
-		(at 118.11 92.71)
-	)
-	(no_connect
-		(at 118.11 80.01)
 	)
 	(no_connect
@@
 	)
 	(no_connect
-		(at 118.11 138.43)
+		(at 118.11 113.03)
 	)
 	(no_connect
-		(at 118.11 113.03)
+		(at 151.13 62.23)
 	)
 	(no_connect
-		(at 118.11 95.25)
+		(at 118.11 85.09)
+	)
+	(no_connect
+		(at 151.13 64.77)
+	)
+	(no_connect
+		(at 118.11 105.41)
 	)
 	(no_connect
@@
 	)
 	(no_connect
-		(at 118.11 135.89)
+		(at 118.11 102.87)
 	)
 	(wire
@@
 	(wire
 		(pts
+			(xy 151.13 69.85) (xy 158.75 69.85)
+		)
+		(stroke
+			(width 0)
+			(type default)
+		)
+	)
+	(wire
+		(pts
 			(xy 176.53 125.73) (xy 184.15 125.73)
 		)
@@
 		(pts
 			(xy 162.56 87.63) (xy 162.56 90.17)
+		)
+		(stroke
+			(width 0)
+			(type default)
+		)
+	)
+	(wire
+		(pts
+			(xy 151.13 67.31) (xy 158.75 67.31)
 		)
 		(stroke
@@
 		)
 	)
+	(label "UART_TX"
+		(at 158.75 67.31 180)
+		(fields_autoplaced yes)
+		(effects
+			(font
+				(size 1.27 1.27)
+			)
+			(justify right bottom)
+		)
+	)
 	(label "~{RST}"
 		(at 177.8 63.5 0)
@@
 			)
 			(justify left bottom)
+		)
+	)
+	(label "UART_RX"
+		(at 158.75 69.85 180)
+		(fields_autoplaced yes)
+		(effects
+			(font
+				(size 1.27 1.27)
+			)
+			(justify right bottom)
 		)
 	)
@@
 	(hierarchical_label "VDMON"
 		(shape input)
-		(at 151.13 64.77 0)
+		(at 151.13 77.47 0)
 		(fields_autoplaced yes)
 		(effects
@@
 	(hierarchical_label "IDMON"
 		(shape input)
-		(at 118.11 105.41 180)
+		(at 151.13 80.01 0)
+		(fields_autoplaced yes)
+		(effects
+			(font
+				(size 1.27 1.27)
+			)
+			(justify left)
+		)
+	)
+	(hierarchical_label "SGOOD"
+		(shape input)
+		(at 118.11 135.89 180)
 		(fields_autoplaced yes)
 		(effects
@@
 	(hierarchical_label "VCTRL"
 		(shape output)
-		(at 151.13 67.31 0)
+		(at 151.13 72.39 0)
 		(fields_autoplaced yes)
 		(effects
@@
 	(hierarchical_label "ICTRL"
 		(shape output)
-		(at 151.13 72.39 0)
+		(at 151.13 74.93 0)
 		(fields_autoplaced yes)
 		(effects
@@
 			)
 			(justify left)
+		)
+	)
+	(hierarchical_label "REG_ON"
+		(shape input)
+		(at 118.11 130.81 180)
+		(fields_autoplaced yes)
+		(effects
+			(font
+				(size 1.27 1.27)
+			)
+			(justify right)
 		)
 	)
 	(hierarchical_label "ISMON"
 		(shape input)
-		(at 118.11 102.87 180)
+		(at 118.11 128.27 180)
 		(fields_autoplaced yes)
 		(effects
@@
 		)
 	)
-	(hierarchical_label "LOAD_DISCHRG"
-		(shape output)
-		(at 118.11 85.09 180)
+	(hierarchical_label "~{FAULT}"
+		(shape input)
+		(at 118.11 138.43 180)
 		(fields_autoplaced yes)
 		(effects
@@
 	(hierarchical_label "SYNC"
 		(shape output)
-		(at 118.11 100.33 180)
+		(at 118.11 123.19 180)
 		(fields_autoplaced yes)
 		(effects
@@
 		)
 	)
-	(hierarchical_label "LOADEN"
-		(shape output)
-		(at 118.11 87.63 180)
+	(hierarchical_label "~{PGOOD}"
+		(shape input)
+		(at 118.11 133.35 180)
 		(fields_autoplaced yes)
 		(effects
@@
 	(hierarchical_label "VSMON"
 		(shape input)
-		(at 151.13 62.23 0)
-		(fields_autoplaced yes)
-		(effects
-			(font
-				(size 1.27 1.27)
-			)
-			(justify left)
+		(at 118.11 80.01 180)
+		(fields_autoplaced yes)
+		(effects
+			(font
+				(size 1.27 1.27)
+			)
+			(justify right)
 		)
 	)
@@
 			)
 			(justify left)
+		)
+	)
+	(hierarchical_label "LOAD_EN"
+		(shape output)
+		(at 118.11 92.71 180)
+		(fields_autoplaced yes)
+		(effects
+			(font
+				(size 1.27 1.27)
+			)
+			(justify right)
+		)
+	)
+	(hierarchical_label "LOAD_DISCHRG"
+		(shape output)
+		(at 118.11 90.17 180)
+		(fields_autoplaced yes)
+		(effects
+			(font
+				(size 1.27 1.27)
+			)
+			(justify right)
+		)
+	)
+	(hierarchical_label "SOURCE_EN"
+		(shape output)
+		(at 118.11 95.25 180)
+		(fields_autoplaced yes)
+		(effects
+			(font
+				(size 1.27 1.27)
+			)
+			(justify right)
+		)
+	)
+	(symbol
+		(lib_id "Connector:TestPoint_Small")
+		(at 118.11 123.19 0)
+		(unit 1)
+		(exclude_from_sim no)
+		(in_bom yes)
+		(on_board yes)
+		(dnp no)
+		(property "Reference" "TP9"
+			(at 116.078 120.396 0)
+			(effects
+				(font
+					(size 1.27 1.27)
+				)
+				(justify left)
+			)
+		)
+		(property "Value" "TestPoint_Small"
+			(at 119.38 124.4599 0)
+			(effects
+				(font
+					(size 1.27 1.27)
+				)
+				(justify left)
+				(hide yes)
+			)
+		)
+		(property "Footprint" "TestPoint:TestPoint_Pad_D1.0mm"
+			(at 123.19 123.19 0)
+			(effects
+				(font
+					(size 1.27 1.27)
+				)
+				(hide yes)
+			)
+		)
+		(property "Datasheet" "~"
+			(at 123.19 123.19 0)
+			(effects
+				(font
+					(size 1.27 1.27)
+				)
+				(hide yes)
+			)
+		)
+		(property "Description" ""
+			(at 118.11 123.19 0)
+			(effects
+				(font
+					(size 1.27 1.27)
+				)
+				(hide yes)
+			)
+		)
+		(pin "1"
+		)
+		(instances
+			(project "PD Charger"
+				(path "/2223e2d2-71c8-4f08-b970-c0182a3b98e5/784b7380-2a85-4f04-b109-d366b8257d5a"
+					(reference "TP9")
+					(unit 1)
+				)
+			)
 		)
 	)
@@
 		)
 		(pin "10"
+			(alternate "LPUART1_TX")
 		)
 		(pin "11"
+			(alternate "LPUART1_RX")
 		)
 		(pin "12"
+			(alternate "DAC1_OUT1")
 		)
 		(pin "13"
+			(alternate "DAC1_OUT2")
 		)
 		(pin "14"
+			(alternate "ADC2_IN3")
 		)
 		(pin "15"
+			(alternate "ADC2_IN4")
 		)
 		(pin "16"
+			(alternate "ADC2_IN5")
 		)
 		(pin "17"
@@
 		)
 		(pin "24"
+			(alternate "ADC1_IN14")
 		)
 		(pin "25"
@@
 		)
 		(pin "30"
+			(alternate "I2C2_SDA")
 		)
 		(pin "31"
+			(alternate "I2C2_SCL")
 		)
 		(pin "32"
 		)
 		(pin "33"
+			(alternate "USB_DM")
 		)
 		(pin "34"
+			(alternate "USB_DP")
 		)
 		(pin "35"
 		)
 		(pin "36"
+			(alternate "SYS_JTMS-SWDIO")
 		)
 		(pin "37"
+			(alternate "SYS_JTCK-SWCLK")
 		)
 		(pin "38"
@@
 		)
 		(pin "41"
+			(alternate "SYS_JTDO-SWO")
 		)
 		(pin "42"
+			(alternate "UCPD1_CC2")
 		)
 		(pin "43"
 		)
 		(pin "44"
+			(alternate "UCPD1_CC1")
 		)
 		(pin "45"
@@
 		)
 		(pin "47"
+			(alternate "TIM17_CH1")
 		)
 		(pin "48"
@@
 					(unit 1)
 				)
-			)
-		)
-	)
-	(symbol
-		(lib_id "Connector:TestPoint_Small")
-		(at 118.11 100.33 0)
-		(unit 1)
-		(exclude_from_sim no)
-		(in_bom yes)
-		(on_board yes)
-		(dnp no)
-		(property "Reference" "TP9"
-			(at 116.078 97.536 0)
-			(effects
-				(font
-					(size 1.27 1.27)
-				)
-				(justify left)
-			)
-		)
-		(property "Value" "TestPoint_Small"
-			(at 119.38 101.5999 0)
-			(effects
-				(font
-					(size 1.27 1.27)
-				)
-				(justify left)
-				(hide yes)
-			)
-		)
-		(property "Footprint" "TestPoint:TestPoint_Pad_D1.0mm"
-			(at 123.19 100.33 0)
-			(effects
-				(font
-					(size 1.27 1.27)
-				)
-				(hide yes)
-			)
-		)
-		(property "Datasheet" "~"
-			(at 123.19 100.33 0)
-			(effects
-				(font
-					(size 1.27 1.27)
-				)
-				(hide yes)
-			)
-		)
-		(property "Description" ""
-			(at 118.11 100.33 0)
-			(effects
-				(font
-					(size 1.27 1.27)
-				)
-				(hide yes)
-			)
-		)
-		(pin "1"
-		)
-		(instances
-			(project "PD Charger"
-				(path "/2223e2d2-71c8-4f08-b970-c0182a3b98e5/784b7380-2a85-4f04-b109-d366b8257d5a"
-					(reference "TP9")
-					(unit 1)
-				)

Commit message: multi sheet redesign
Connections:
- no-connect marks 13 -> 14
Changed lines of the file:
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@@
+	)
+	(no_connect
+		(at 118.11 100.33)
 	)
 	(no_connect

Commit message: standalone regulator core
Parts:
- J2: footprint Connector:Tag-Connect_TC2030-IDC-NL_2x03_P1.27mm_Vertical -> Connector:Tag-Connect_TC2030-IDC-FP_2x03_P1.27mm_Vertical
Changed lines of the file:
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@@
 			)
 		)
-		(property "Description" ""
+		(property "Description" "test point"
 			(at 118.11 123.19 0)
 			(effects
@@
 			)
 		)
-		(property "Description" ""
+		(property "Description" "Unpolarized capacitor"
 			(at 191.77 129.54 0)
 			(effects
@@
 			)
 		)
-		(property "Description" ""
+		(property "Description" "Unpolarized capacitor"
 			(at 109.22 66.04 0)
 			(effects
@@
 			)
 		)
-		(property "Description" ""
+		(property "Description" "Power symbol creates a global label with name \"GND\" , ground"
 			(at 95.25 142.24 0)
 			(effects
@@
 			)
 		)
-		(property "Description" ""
+		(property "Description" "Unpolarized capacitor"
 			(at 176.53 129.54 0)
 			(effects
@@
 			)
 		)
-		(property "Description" ""
+		(property "Description" "Power symbol creates a global label with name \"GND\" , ground"
 			(at 170.18 133.35 0)
 			(effects
@@
 			)
 		)
-		(property "Description" ""
+		(property "Description" "Power symbol creates a global label with name \"+3V3\""
 			(at 100.33 78.74 0)
 			(effects
@@
 			)
 		)
-		(property "Description" ""
+		(property "Description" "STMicroelectronics Arm Cortex-M4 MCU, 32KB flash, 32KB RAM, 170 MHz, 1.71-3.6V, 42 GPIO, UFQFPN48"
 			(at 133.35 102.87 0)
 			(effects
@@
 			)
 		)
-		(property "Footprint" "Connector:Tag-Connect_TC2030-IDC-NL_2x03_P1.27mm_Vertical"
+		(property "Footprint" "Connector:Tag-Connect_TC2030-IDC-FP_2x03_P1.27mm_Vertical"
 			(at 189.23 86.36 0)
 			(effects
@@
 			)
 		)
-		(property "Description" ""
+		(property "Description" "Tag-Connect ARM Cortex SWD JTAG connector, 6 pin"
 			(at 189.23 68.58 0)
 			(effects
@@
 			)
 		)
-		(property "Description" ""
+		(property "Description" "Unpolarized capacitor"
 			(at 184.15 129.54 0)
 			(effects
@@
 			)
 		)
-		(property "Description" ""
+		(property "Description" "Unpolarized capacitor"
 			(at 170.18 129.54 0)
 			(effects
@@
 			)
 		)
-		(property "Description" ""
+		(property "Description" "Resistor"
 			(at 100.33 82.55 0)
 			(effects
@@
 			)
 		)
-		(property "Description" ""
+		(property "Description" "Power symbol creates a global label with name \"+3V3\""
 			(at 191.77 58.42 0)
 			(effects
@@
 			)
 		)
-		(property "Description" ""
+		(property "Description" "Unpolarized capacitor"
 			(at 100.33 90.17 0)
 			(effects
@@
 			)
 		)
-		(property "Description" ""
+		(property "Description" "Power symbol creates a global label with name \"GND\" , ground"
 			(at 135.89 146.05 0)
 			(effects
@@
 			)
 		)
-		(property "Description" ""
+		(property "Description" "Power symbol creates a global label with name \"+3V3\""
 			(at 130.81 57.15 0)
 			(effects
@@
 			)
 		)
-		(property "Description" ""
+		(property "Description" "Power symbol creates a global label with name \"GND\" , ground"
 			(at 93.98 96.52 0)
 			(effects
@@
 			)
 		)
-		(property "Description" ""
+		(property "Description" "Solder Jumper, 2-pole, open"
 			(at 165.1 91.44 0)
 			(effects
@@
 			)
 		)
-		(property "Description" ""
+		(property "Description" "Power symbol creates a global label with name \"GND\" , ground"
 			(at 191.77 78.74 0)
 			(effects
@@
 			)
 		)
-		(property "Description" ""
+		(property "Description" "Resistor"
 			(at 95.25 138.43 0)
 			(effects
@@
 			)
 		)
-		(property "Description" ""
+		(property "Description" "Power symbol creates a global label with name \"+3V3\""
 			(at 170.18 125.73 0)
 			(effects
@@
 			)
 		)
-		(property "Description" ""
+		(property "Description" "Push button switch, generic, two pins"
 			(at 95.25 129.54 0)
 			(effects
@@
 			)
 		)
-		(property "Description" ""
+		(property "Description" "Power symbol creates a global label with name \"GND\" , ground"
 			(at 109.22 69.85 0)
 			(effects
@@
 			)
 		)
-		(property "Description" ""
+		(property "Description" "Unpolarized capacitor"
 			(at 199.39 129.54 0)
 			(effects
@@
 			)
 		)
-		(property "Description" ""
+		(property "Description" "Push button switch, generic, two pins"
 			(at 93.98 91.44 0)
 			(effects
